Commit message: v0.1

File: curiosity/urdf/curiocity.xacro (robot description, xacro)
@@ -1,456 +1,247 @@
 <?xml version="1.0"?>
 <robot name="curiosity_rover" xmlns:xacro="http://www.ros.org/wiki/xacro">
+<xacro:property name="ll" value="link_left"/>
+<xacro:property name="lr" value="link_right"/>
+<xacro:property name="roboname" value="curiosity_rover"/>
+<xacro:property name="base_length" value="2.7"/>
+<xacro:property name="base_width" value="5"/>
+<xacro:property name="base_height" value="1"/>
+<xacro:property name="base_x" value="0"/>
+<xacro:property name="base_y" value="0"/>
+<xacro:property name="base_z" value="2"/>
+<!--Base link-->
 <link name="base_link">
-	    <inertial>
-	      <mass value="20.3" />
-	      <origin xyz="0 0 0.0" />
-	      <inertia ixx="0.07" ixy="0.0" ixz="0.0"
-	        iyy="0.08" iyz="0.00" izz="0.10" />
-	    </inertial>
-	    <visual>
-		<origin xyz="0 0 0" rpy="0 0 0" />
-	      <geometry>
-		<box size="1 1 1" />
-	      </geometry>
-		<material name="red" />
-	    </visual>
-	    <collision>
-	      <origin xyz="0.00 0.0 0.0" rpy="0 0 0" />
-	      <geometry>
-	         <box size="1 1 1" />
-	      </geometry>
-	    </collision>
-</link>
-	    <!--Left-Back-->
-<link name="link-left-back">
-	    <inertial>
-	      <mass value="5.3" />
-	      <origin xyz="0 0 0.0" />
-	      <inertia ixx="0.07" ixy="0.0" ixz="0.0"
-	        iyy="0.08" iyz="0.00" izz="0.10" />
-	    </inertial>
-	    <visual>
-		<origin xyz="2 5 6" rpy="0 0 0" />
-	      <geometry>
-		<box size="1 1 1" />
-	      </geometry>
-		<material name="red" />
-	    </visual>
-	    <collision>
-	      <origin xyz="0.00 0.0 0.0" rpy="0 0 0" />
-	      <geometry>
-	         <box size="1 1 1" />
-	      </geometry>
-	    </collision>
-</link>
-<!--Left-Back1-->
-<link name="Link-Left-Back1">
-	    <inertial>
-	      <mass value="2.3" />
-	      <origin xyz="0 0 0.0" />
-	      <inertia ixx="0.07" ixy="0.0" ixz="0.0"
-	        iyy="0.08" iyz="0.00" izz="0.10" />
-	    </inertial>
-	    <visual>
-		<origin xyz="0 0 0" rpy="0 0 0" />
-	      <geometry>
-		<box size="1 1 1" />
-	      </geometry>
-		<material name="red" />
-	    </visual>
-	    <collision>
-	      <origin xyz="0.00 0.0 0.0" rpy="0 0 0" />
-	      <geometry>
-	         <box size="1 1 1" />
-	      </geometry>
-	    </collision>
-</link>
-<!--Left-Back1-Wheel-->
-<link name="Link-Left-Back1-Wheel">
-	    <inertial>
-	      <mass value="7" />
-	      <origin xyz="0 0 0.0" />
-	      <inertia ixx="0.07" ixy="0.0" ixz="0.0"
-	        iyy="0.08" iyz="0.00" izz="0.10" />
-	    </inertial>
-	    <visual>
-		<origin xyz="0 0 0" rpy="0 0 0" />
-	      <geometry>
-		<box size="1 1 1" />
-	      </geometry>
-		<material name="red" />
-	    </visual>
-	    <collision>
-	      <origin xyz="0.00 0.0 0.0" rpy="0 0 0" />
-	      <geometry>
-	         <box size="1 1 1" />
-	      </geometry>
-	    </collision>
-</link>
-<!--Left-Back2-->
-<link name="Link-Left-Back2">
-	    <inertial>
-	      <mass value="2.3" />
-	      <origin xyz="0 0 0.0" />
-	      <inertia ixx="0.07" ixy="0.0" ixz="0.0"
-	        iyy="0.08" iyz="0.00" izz="0.10" />
-	    </inertial>
-	    <visual>
-		<origin xyz="0 0 0" rpy="0 0 0" />
-	      <geometry>
-		<box size="1 1 1" />
-	      </geometry>
-		<material name="red" />
-	    </visual>
-	    <collision>
-	      <origin xyz="0.00 0.0 0.0" rpy="0 0 0" />
-	      <geometry>
-	         <box size="1 1 1" />
-	      </geometry>
-	    </collision>
-</link>
-<!-- Left-Back2-wheel -->
-<link name="Link-Left-Back2-wheel">
-	    <inertial>
-	      <mass value="7" />
-	      <origin xyz="0 0 0.0" />
-	      <inertia ixx="0.07" ixy="0.0" ixz="0.0"
-	        iyy="0.08" iyz="0.00" izz="0.10" />
-	    </inertial>
-	    <visual>
-		<origin xyz="0 0 0" rpy="0 0 0" />
-	      <geometry>
-		<box size="1 1 1" />
-	      </geometry>
-		<material name="red" />
-	    </visual>
-	    <collision>
-	      <origin xyz="0.00 0.0 0.0" rpy="0 0 0" />
-	      <geometry>
-	         <box size="1 1 1" />
-	      </geometry>
-	    </collision>
-</link>
-<!--Left-Front-->
-<link name="Link-Left-Front">
-	    <inertial>
-	      <mass value="5.3" />
-	      <origin xyz="0 0 0.0" />
-	      <inertia ixx="0.07" ixy="0.0" ixz="0.0"
-	        iyy="0.08" iyz="0.00" izz="0.10" />
-	    </inertial>
-	    <visual>
-		<origin xyz="0 0 0" rpy="0 0 0" />
-	      <geometry>
-		<box size="1 1 1" />
-	      </geometry>
-		<material name="red" />
-	    </visual>
-	    <collision>
-	      <origin xyz="0.00 0.0 0.0" rpy="0 0 0" />
-	      <geometry>
-	         <box size="1 1 1" />
-	      </geometry>
-	    </collision>
-</link>
-<!-- Left-Front-Wheel -->
-<link name="Link-Left-Front-Wheel">
-	    <inertial>
-	      <mass value="7" />
-	      <origin xyz="0 0 0.0" />
-	      <inertia ixx="0.07" ixy="0.0" ixz="0.0"
-	        iyy="0.08" iyz="0.00" izz="0.10" />
-	    </inertial>
-	    <visual>
-		<origin xyz="0 0 0" rpy="0 0 0" />
-	      <geometry>
-		<box size="1 1 1" />
-	      </geometry>
-		<material name="red" />
-	    </visual>
-	    <collision>
-	      <origin xyz="0.00 0.0 0.0" rpy="0 0 0" />
-	      <geometry>
-	         <box size="1 1 1" />
-	      </geometry>
-	    </collision>
-</link>
-<!-- Camera-Base -->
-<link name="Link-Camera-Base">
-	    <inertial>
-	      <mass value="2.5" />
-	      <origin xyz="0 0 0.0" />
-	      <inertia ixx="0.07" ixy="0.0" ixz="0.0"
-	        iyy="0.08" iyz="0.00" izz="0.10" />
-	    </inertial>
-	    <visual>
-		<origin xyz="0 0 0" rpy="0 0 0" />
-	      <geometry>
-		<box size="1 1 1" />
-	      </geometry>
-		<material name="red" />
-	    </visual>
-	    <collision>
-	      <origin xyz="0.00 0.0 0.0" rpy="0 0 0" />
-	      <geometry>
-	         <box size="1 1 1" />
-	      </geometry>
-	    </collision>
-</link>
-<!-- Camera -->
-<link name="Camera">
-	    <inertial>
-	      <mass value="1.5" />
-	      <origin xyz="0 0 0.0" />
-	      <inertia ixx="0.07" ixy="0.0" ixz="0.0"
-	        iyy="0.08" iyz="0.00" izz="0.10" />
-	    </inertial>
-	    <visual>
-		<origin xyz="0 0 0" rpy="0 0 0" />
-	      <geometry>
-		<box size="1 1 1" />
-	      </geometry>
-		<material name="red" />
-	    </visual>
-	    <collision>
-	      <origin xyz="0.00 0.0 0.0" rpy="0 0 0" />
-	      <geometry>
-	         <box size="1 1 1" />
-	      </geometry>
-	    </collision>
-</link>
-<!--Right-Back-->
-<link name="Link-Right-Back">
-	    <inertial>
-	      <mass value="5.3" />
-	      <origin xyz="0 0 0.0" />
-	      <inertia ixx="0.07" ixy="0.0" ixz="0.0"
-	        iyy="0.08" iyz="0.00" izz="0.10" />
-	    </inertial>
-	    <visual>
-		<origin xyz="0 0 0" rpy="0 0 0" />
-	      <geometry>
-		<box size="1 1 1" />
-	      </geometry>
-		<material name="red" />
-	    </visual>
-	    <collision>
-	      <origin xyz="0.00 0.0 0.0" rpy="0 0 0" />
-	      <geometry>
-	         <box size="1 1 1" />
-	      </geometry>
-	    </collision>
-	    <!--Right-Back1-->
-</link>
-<link name="Link-Right-Back1">
-	    <inertial>
-	      <mass value="2.3" />
-	      <origin xyz="0 0 0.0" />
-	      <inertia ixx="0.07" ixy="0.0" ixz="0.0"
-	        iyy="0.08" iyz="0.00" izz="0.10" />
-	    </inertial>
-	    <visual>
-		<origin xyz="0 0 0" rpy="0 0 0" />
-	      <geometry>
-		<box size="1 1 1" />
-	      </geometry>
-		<material name="red" />
-	    </visual>
-	    <collision>
-	      <origin xyz="0.00 0.0 0.0" rpy="0 0 0" />
-	      <geometry>
-	         <box size="1 1 1" />
-	      </geometry>
-	    </collision>
-	    <!--Right-Back1-Wheel-->
-</link>
-<link name="Link-Right-Back1-Wheel">
-	    <inertial>
-	      <mass value="7" />
-	      <origin xyz="0 0 0.0" />
-	      <inertia ixx="0.07" ixy="0.0" ixz="0.0"
-	        iyy="0.08" iyz="0.00" izz="0.10" />
-	    </inertial>
-	    <visual>
-		<origin xyz="0 0 0" rpy="0 0 0" />
-	      <geometry>
-		<box size="1 1 1" />
-	      </geometry>
-		<material name="red" />
-	    </visual>
-	    <collision>
-	      <origin xyz="0.00 0.0 0.0" rpy="0 0 0" />
-	      <geometry>
-	         <box size="1 1 1" />
-	      </geometry>
-	    </collision>
-</link>
-<!--Right-Back2-->
-<link name="Link-Right-Back2">
-	    <inertial>
-	      <mass value="2.3" />
-	      <origin xyz="0 0 0.0" />
-	      <inertia ixx="0.07" ixy="0.0" ixz="0.0"
-	        iyy="0.08" iyz="0.00" izz="0.10" />
-	    </inertial>
-	    <visual>
-		<origin xyz="0 0 0" rpy="0 0 0" />
-	      <geometry>
-		<box size="1 1 1" />
-	      </geometry>
-		<material name="red" />
-	    </visual>
-	    <collision>
-	      <origin xyz="0.00 0.0 0.0" rpy="0 0 0" />
-	      <geometry>
-	         <box size="1 1 1" />
-	      </geometry>
-	    </collision>
-	    <!-- Right-Back2-wheel -->
-</link>
-<link name="Link-Right-Back2-wheel">
-	    <inertial>
-	      <mass value="7" />
-	      <origin xyz="0 0 0.0" />
-	      <inertia ixx="0.07" ixy="0.0" ixz="0.0"
-	        iyy="0.08" iyz="0.00" izz="0.10" />
-	    </inertial>
-	    <visual>
-		<origin xyz="0 0 0" rpy="0 0 0" />
-	      <geometry>
-		<box size="1 1 1" />
-	      </geometry>
-		<material name="red" />
-	    </visual>
-	    <collision>
-	      <origin xyz="0.00 0.0 0.0" rpy="0 0 0" />
-	      <geometry>
-	         <box size="1 1 1" />
-	      </geometry>
-	    </collision>
-</link>
-<!--Right-Front-->
-<link name="Link-Right-Front">
-	    <inertial>
-	      <mass value="5.3" />
-	      <origin xyz="0 0 0.0" />
-	      <inertia ixx="0.07" ixy="0.0" ixz="0.0"
-	        iyy="0.08" iyz="0.00" izz="0.10" />
-	    </inertial>
-	    <visual>
-		<origin xyz="0 0 0" rpy="0 0 0" />
-	      <geometry>
-		<box size="1 1 1" />
-	      </geometry>
-		<material name="red" />
-	    </visual>
-	    <collision>
-	      <origin xyz="0.00 0.0 0.0" rpy="0 0 0" />
-	      <geometry>
-	         <box size="1 1 1" />
-	      </geometry>
-	    </collision>
-	    <!-- Right-Front-Wheel -->
-</link>
-<link name="link_right_wheel">
-	    <inertial>
-	      <mass value="7" />
-	      <origin xyz="0 0 0.0" />
-	      <inertia ixx="0.07" ixy="0.0" ixz="0.0"
-	        iyy="0.08" iyz="0.00" izz="0.10" />
-	    </inertial>
-	    <visual>
-		<origin xyz="0 0 0" rpy="0 0 0" />
-	      <geometry>
-		<box size="1 1 1" />
-	      </geometry>
-		<material name="red" />
-	    </visual>
-	    <collision>
-	      <origin xyz="0.00 0.0 0.0" rpy="0 0 0" />
-	      <geometry>
-	         <box size="1 1 1" />
-	      </geometry>
-	    </collision>
-</link>
-<joint name="joint_left_wheels" type="fixed">
-<parent link="base_link"/>
-<child link= "link-left-back"/>
-<origin rpy="0 -0 0" xyz="-3 -4 6"/>
-</joint>
-<joint name="joint_left_wheels6" type="fixed">
-<parent link="base_link"/>
-<child link= "Link-Camera-Base"/>
-<origin rpy="0 -0 0" xyz="-3 -4 6"/>
-</joint>
-<joint name="joint_left_wheels7" type="fixed">
-<parent link="Link-Camera-Base"/>
-<child link= "Camera"/>
-<origin rpy="0 -0 0" xyz="-3 -4 6"/>
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